File: kicad/bal02/bal02.kicad_sch (KiCad schematic)
At the start: 4 parts, among them IC1 nucleo32-L432, IC2 nRF24L01_SMD_MODULE, IC3 MPU9250_SMD_MODULE

Commit message: more components added
Parts:
- added C1, C2: C, symbol Device:C
- added C3, C4: 100uF/25V, bal:WCAP-ATG8, symbol Device:C_Polarized
- added D2, D3: 1N4148WT, Diode_SMD:D_SOD-523, symbol Diode:1N4148WT
- added IC4: M24C16-FMN6TP, bal:SOIC127P600X175-8N, symbol bal_symbols:M24C16-FMN6TP
- added IC5: SN65HVD230DR, bal:SOT127P600X175-8N, symbol bal_symbols:SN65HVD230DR
- added IC6: TLV76050DBZR, bal:SOT95P237X112-3N, symbol bal_symbols:TLV76050DBZR
- added R1, R2, R3, R4: R, symbol Device:R
- added R5, R6: 4k7, symbol Device:R
Connections:
- net +3V3: now also IC4.7 (~{WC}), IC4.8 (VCC), R5.1, R6.1
- net +5V: now also C2.1, IC6.1 (OUT)
- net ACC_MISO: now also R4.1
- net ACC_MOSI: now also R3.1
- net GND: now also C1.2, C2.2, C3.2, C4.2, IC4.4 (VSS), IC6.3 (GND)
- net I2C1_SCL: now also IC4.6 (SCL), R5.2
- net I2C1_SDA: now also IC4.5 (SDA), R6.2
- net nRF_MISO: now also R2.1; no longer IC2.7 (MISO)
- net nRF_MOSI: now also R1.1; no longer IC2.6 (MOSI)
- net at IC3.4 (SDA): now also R3.2
- net at IC3.7 (AD0): now also R4.2
- new net: C1.1, C3.1, C4.1, D2.1 (K), D3.1 (K), IC6.2 (IN)
- new net: IC2.6 (MOSI), R1.2
- new net: IC2.7 (MISO), R2.2
- no-connect marks 0 -> 12
Other:
- note added: "860010473007"

Commit message: bal02 placement + nucleo32 update
Parts:
- added C1: 10uF, Capacitor_SMD:C_0805_2012Metric, symbol Device:C
- added C5, C6: 100nF, Capacitor_SMD:C_0603_1608Metric, symbol Device:C
- added R10, R9: R, Resistor_SMD:R_0402_1005Metric, symbol Device:R
- added R7: 0R, Resistor_SMD:R_0603_1608Metric, symbol Device:R
- added R8: 120R, Resistor_SMD:R_0603_1608Metric, symbol Device:R
- added X1, X2, X3, X5: ~, bal:H2_100mil, symbol bal_symbols:H2_100mil
- added X4, X6: ~, bal:H4_50mil, symbol bal_symbols:H4_50mil
- C2: value C -> 100nF; footprint (none) -> Capacitor_SMD:C_0603_1608Metric
- C7: renamed from C1; value C -> 100nF; footprint (none) -> Capacitor_SMD:C_0603_1608Metric
- R1, R2, R3, R4: footprint (none) -> Resistor_SMD:R_0402_1005Metric
- R5, R6: footprint (none) -> Resistor_SMD:R_0603_1608Metric
Connections:
- net +3V3: now also IC5.3 (VCC), C5.1, C6.1
- net +5V: now also R10.1, R9.1
- net CAN_RX: now also IC5.4 (R)
- net CAN_TX: now also IC5.1 (D)
- net GND: now also IC5.2 (GND), C1.2, C5.2, C6.2, R7.2, X1.2, X2.2, X3.2, X4.4, X5.2, X6.4
- net +BATT: now reaches C3.1, C4.1, C7.1, D2.1 (K), D3.1 (K), IC6.2 (IN)
- net +BATT: now also C1.1, X3.1, X5.1
- net at IC5.6 (CANL): now also R8.2, X4.3, X6.3
- net at IC5.7 (CANH): now also R8.1, X4.2, X6.2
- net at IC5.8 (RS): now also R7.1
- net at D3.2 (A): now also X2.1
- net at D2.2 (A): now also X1.1
- new net: R10.2, X6.1
- new net: R9.2, X4.1
- no-connect marks 12 -> 13
Other:
- note added: "+5V CAN_H CAN_L GND"
- note added: "Bat1"
- note added: "Bat2"
- note added: "Motor 1"
- note added: "Motor 2"
- note added: "VBat GND"
- note removed: "+5V CAN TX/RX GND"
- note removed: "2 x large CAP"
- note removed: "5V DCD/LDO"
- note removed: "I2C EEPROM"
- moved on the sheet: C3, C7, D2, D3, IC5
